File: USB2XXX.kicad_sch (KiCad schematic)
At the start: 12 parts, among them J1 Conn_01x04, J2 Conn_01x03, J3 Conn_01x03, J4 Conn_01x02, J5 Conn_01x02

Commit message: Big update on UART-pilot lamp/routings/connectors/esd protection
Parts:
- added H1, H2, H3, H4: MountingHole, MountingHole:MountingHole_2.7mm_M2.5, symbol Mechanical:MountingHole
- D8: value LED -> GREEN
- J3: value Conn_01x03 -> Conn_01x02; footprint Connector_JST:JST_GH_SM03B-GHS-TB_1x03-1MP_P1.25mm_Horizontal -> Connector:MountingHole_0.8mm_sm2.5_2pin; symbol Connector_Generic:Conn_01x03 -> Connector_Generic:Conn_01x02
- J4, J5: footprint Connector_JST:JST_GH_SM02B-GHS-TB_1x02-1MP_P1.25mm_Horizontal -> Connector:MountingHole_0.8mm_sm2.5_2pin
Connections:
- net GND: no longer J3.3 (Pin_3)
